File: docs/engineering/rvb22/candidate/cad/GR86_CCA_RevB.kicad_pcb (KiCad board)
At the start: 4 copper layers, 88.3 x 61.3 mm, 199 parts, among them J201 TC2030-IDC-NL / UART, J202 RESET — short to reset, J203 BOOT — hold low on reset, J401 U.FL-R-SMT-1(80), Q101 STD25NF20 /200V, U101 LTC4367HMS8#WTRPBF, U121 LM5164DDAR, U151 LM63615DQPWPRQ1, U201 ESP32-S3-WROOM-1-N8R2, U202 TPS3808G33-Q1 3.07V RESET, U301 TCAN3403DRBRQ1, U401 PA1616D, U402 SN74LVC2G125DCUR, U403 MIC5504-3.3YM5-TR, U404 SN74LVC2G125DCUR, U501 TPS26600PWPR, U502 OPA2333AIDR

Commit message: fix(cca): reconcile controlled footprint variants and retain coupled thermal redlines
Parts:
- C154: footprint RevB:C_0603_1608Metric -> RevB:C_0603_1608Metric_RVB22_C154
- C205: footprint RevB:C_0603_1608Metric -> RevB:C_0603_1608Metric_RVB22_C205
- C206: footprint RevB:KEMET_T598_X_7343_Median -> RevB:KEMET_T598_X_7343_Median_RVB22_C206
- D103: footprint RevB:D_SMC -> RevB:D_SMC_RVB22_D103
- F1: footprint RevB:Molex_Micro-Fit_3.0_43045-1200_2x06_P3.00mm_Horizontal -> RevB:Molex_Micro-Fit_3.0_43045-1200_2x06_P3.00mm_Horizontal_RVB22_F1
- L121: footprint RevB:Coilcraft_MSS1246T_12x12 -> RevB:Coilcraft_MSS1246T_12x12_RVB22_L121
- R155: footprint RevB:R_0603_1608Metric -> RevB:R_0603_1608Metric_RVB22_R155
- R156: footprint RevB:R_0603_1608Metric -> RevB:R_0603_1608Metric_RVB22_R156
- R157: footprint RevB:R_0603_1608Metric -> RevB:R_0603_1608Metric_RVB22_R157
- R203: footprint RevB:R_0603_1608Metric -> RevB:R_0603_1608Metric_RVB22_R203
- U151: footprint RevB:HTSSOP-16-1EP_4.4x5mm_P0.65mm_EP3.4x5mm_Mask2.46x2.31mm -> RevB:HTSSOP-16-1EP_4.4x5mm_P0.65mm_EP3.4x5mm_Mask2.46x2.31mm_RVB22_U151
- U201: footprint RevB:ESP32-S3-WROOM-1 -> RevB:ESP32-S3-WROOM-1_RVB22_U201
