File: docs/engineering/rvb22/candidate/cad/GR86_CCA_RevB.kicad_pcb (KiCad board)
At the start: 4 copper layers, 88.3 x 61.3 mm, 199 parts, among them J201 TC2030-IDC-NL / UART, J202 RESET — short to reset, J203 BOOT — hold low on reset, J401 U.FL-R-SMT-1(80), Q101 STD25NF20 /200V, U101 LTC4367HMS8#WTRPBF, U121 LM5164DDAR, U151 LM63615DQPWPRQ1, U201 ESP32-S3-WROOM-1-N8R2, U202 TPS3808G33-Q1 3.07V RESET, U301 TCAN3403DRBRQ1, U401 PA1616D, U402 SN74LVC2G125DCUR, U403 MIC5504-3.3YM5-TR, U404 SN74LVC2G125DCUR, U501 TPS26600PWPR, U502 OPA2333AIDR

Commit message: Move C206 onto thermal tab and preserve coordinated I18 redlines
Parts:
- C206: moved to F.Cu
- moved C206 22.4 mm to (82.0, -4.00)
Routing:
- net 3V3_BULK_DAMPED: track 2.54 -> 32.0 mm, vias 0 -> 2
- net GND: track 176.8 -> 179.6 mm, vias 154 -> 156
Other:
- outline, holes or cut-outs redrawn

Commit message: RVB22 I19: tighten 3V3 feedback tolerance and thermal drift allocation
Parts:
- R155: value 23.7k /0.1% 25ppm FB TOP -> 11.8k /0.02% 2ppm FB TOP
- R156: value 10k /0.1% 25ppm FB BOTTOM -> 4.99k /0.02% 2ppm FB BOTTOM

Commit message: RVB22 I23: remove LED intrusions from digital reference paths
Routing:
- net LED_CAN: track 77.2 -> 101.1 mm
- net LED_BLE: track 67.9 -> 65.8 mm

Commit message: RVB22 I23: enforce native keepouts and voltage clearances on reroutes
Routing:
- net LED_BLE: track 65.8 -> 82.3 mm
- net LED_CAN: track 101.1 -> 113.8 mm

Commit message: I24: shorten oil routes to restore CAN RX reference paths
Routing:
- net OIL_5V: track 97.8 -> 91.1 mm
Changed lines of the file:
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@@
 (segment (start 20.75 28.7) (end 21.75 29.5) (width 0.4) (locked yes) (layer "B.Cu") (net 66))
 (segment (start 68.4 34.5) (end 68.4 36.6788) (width 0.6) (layer "B.Cu") (net 66))
-(segment (start 25.6 25.744) (end 24.5522 25.744) (width 0.4) (locked yes) (layer "In1.Cu") (net 66))
-(segment (start 20.75 30.3) (end 25.6 30.3) (width 0.4) (locked yes) (layer "In1.Cu") (net 66))
-(segment (start 20.75 28.7) (end 20.75 30.3) (width 0.4) (locked yes) (layer "In1.Cu") (net 66))
-(segment (start 25.6 30.3) (end 25.6 25.744) (width 0.4) (locked yes) (layer "In1.Cu") (net 66))
 (segment (start 83.5 28.455) (end 84.2 28.455) (width 0.2) (locked yes) (layer "B.Cu") (net 67))
 (segment (start 80.975 28.595) (end 83.5 28.455) (width 0.2) (locked yes) (layer "B.Cu") (net 67))
@@
 (segment (start 45 38.85) (end 44.95 38.8) (width 0.2) (locked yes) (layer "B.Cu") (net 80))
 (segment (start 47.8 40.2) (end 47.75 40.15) (width 0.2) (locked yes) (layer "B.Cu") (net 80))
-(segment (start 26.2 38.55) (end 26.15 38.55) (width 0.2) (locked yes) (layer "In1.Cu") (net 80))
-(segment (start 25.55 37.95) (end 25.5 37.95) (width 0.2) (locked yes) (layer "In1.Cu") (net 80))
-(segment (start 26.25 38.6) (end 26.2 38.55) (width 0.2) (locked yes) (layer "In1.Cu") (net 80))
-(segment (start 24.85 37.3) (end 21.15 37.3) (width 0.2) (locked yes) (layer "In1.Cu") (net 80))
-(segment (start 25.5 37.95) (end 24.85 37.3) (width 0.2) (locked yes) (layer "In1.Cu") (net 80))
-(segment (start 42.75 38.6) (end 26.25 38.6) (width 0.2) (locked yes) (layer "In1.Cu") (net 80))
-(segment (start 26.15 38.55) (end 25.55 37.95) (width 0.2) (locked yes) (layer "In1.Cu") (net 80))
 (segment (start 11.5185 28.97) (end 11.5185 29.0728) (width 0.2) (layer "F.Cu") (net 81))
 (segment (start 12.3277 28.1608) (end 11.5185 28.97) (width 0.2) (layer "F.Cu") (net 81))
@@
 (segment (start 80.8 15.8) (end 80.8 13.85) (width 0.2) (layer "In2.Cu") (net 56))
 (segment (start 80.8 13.85) (end 79.85 12.9) (width 0.2) (layer "In2.Cu") (net 56))
+(segment (start 20.75 28.7) (end 20.75 28.15) (width 0.4) (layer "In2.Cu") (net 66))
+(segment (start 20.75 28.15) (end 22.0 26.9) (width 0.4) (layer "In2.Cu") (net 66))
+(segment (start 22.0 26.9) (end 23.156 25.744) (width 0.4) (layer "In2.Cu") (net 66))
+(segment (start 23.156 25.744) (end 24.5522 25.744) (width 0.4) (layer "In2.Cu") (net 66))
+(segment (start 21.15 37.3) (end 22.45 38.6) (width 0.2) (layer "In2.Cu") (net 80))
+(segment (start 22.45 38.6) (end 42.75 38.6) (width 0.2) (layer "In2.Cu") (net 80))
 )

Commit message: I24: preserve alternate CAN TX reference through coordinated LED clearance
Routing:
- net LED_CAN: track 113.8 -> 115.8 mm
Changed lines of the file:
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@@
 (segment (start 51.2 27.6) (end 68.4 27.6) (width 0.2) (layer "In2.Cu") (net 56))
 (segment (start 68.4 27.6) (end 79.9 16.1) (width 0.2) (layer "In2.Cu") (net 56))
-(segment (start 79.9 16.1) (end 80.5 16.1) (width 0.2) (layer "In2.Cu") (net 56))
-(segment (start 80.5 16.1) (end 80.8 15.8) (width 0.2) (layer "In2.Cu") (net 56))
-(segment (start 80.8 15.8) (end 80.8 13.85) (width 0.2) (layer "In2.Cu") (net 56))
-(segment (start 80.8 13.85) (end 79.85 12.9) (width 0.2) (layer "In2.Cu") (net 56))
 (segment (start 20.75 28.7) (end 20.75 28.15) (width 0.4) (layer "In2.Cu") (net 66))
 (segment (start 20.75 28.15) (end 22.0 26.9) (width 0.4) (layer "In2.Cu") (net 66))
@@
 (segment (start 21.15 37.3) (end 22.45 38.6) (width 0.2) (layer "In2.Cu") (net 80))
 (segment (start 22.45 38.6) (end 42.75 38.6) (width 0.2) (layer "In2.Cu") (net 80))
+(segment (start 79.9 16.1) (end 80.8 16.1) (width 0.2) (layer "In2.Cu") (net 56))
+(segment (start 80.8 16.1) (end 81.7 15.2) (width 0.2) (layer "In2.Cu") (net 56))
+(segment (start 81.7 15.2) (end 82.2 14.7) (width 0.2) (layer "In2.Cu") (net 56))
+(segment (start 82.2 14.7) (end 82.2 14.1) (width 0.2) (layer "In2.Cu") (net 56))
+(segment (start 82.2 14.1) (end 81.0 12.9) (width 0.2) (layer "In2.Cu") (net 56))
+(segment (start 81.0 12.9) (end 79.85 12.9) (width 0.2) (layer "In2.Cu") (net 56))
 )
