File: docs/engineering/rvb22/candidate/cad/Input_Protection.kicad_sch (KiCad schematic)
At the start: 25 parts, among them Q101 STD25NF20 /200V, U101 LTC4367HMS8#WTRPBF

Commit message: fix(cca): reconcile controlled footprint variants and retain coupled thermal redlines
Parts:
- D103: footprint RevB:D_SMC -> RevB:D_SMC_RVB22_D103
Changed lines of the file:
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@@
 (wire (pts (xy 346.71 55.88) (xy 351.79 55.88)) (stroke (width 0) (type default)))
 (global_label "GND" (shape bidirectional) (at 351.79 55.88 0) (effects (font (size 1.0 1.0)) (justify left)) (property "Intersheetrefs" "${INTERSHEET_REFS}" (at 351.79 55.88 0) (effects (font (size 1.27 1.27)) (justify left) hide)))
-(symbol (lib_id "Device:D_Zener") (at 342.9 55.88 0) (unit 1) (in_bom yes) (on_board yes) (dnp no) (property "Reference" "D103" (at 337.82 46.99 0) (effects (font (size 1.27 1.27)) (justify left))) (property "Value" "SMCJ24A /TVS" (at 337.82 49.53 0) (effects (font (size 1.27 1.27)) (justify left))) (property "Footprint" "RevB:D_SMC" (at 0 0 0) (effects (font (size 1.27 1.27)) (justify left) hide)) (property "Datasheet" "~" (at 0 0 0) (effects (font (size 1.27 1.27)) (justify left) hide)) (property "MPN" "SMCJ24AHE3_A/H" (at 0 0 0) (effects (font (size 1.27 1.27)) (justify left) hide)) (property "Qualification" "VERIFIED component selection; qualification/productization/SELECTED_COMPONENTS.json; physical acceptance separate" (at 0 0 0) (effects (font (size 1.27 1.27)) (justify left) hide)) (pin "1") (pin "2") (instances (project "GR86_CCA_RevB" (path "/4108b523-946e-532e-b734-a3b8d9b0fa0b/33d5571c-9bbc-5869-9406-ade8bba2c66d" (reference "D103") (unit 1)))) (property "Manufacturer" "Vishay" (at 0 0 0) (effects (font (size 1.27 1.27)) (hide yes))) (property "LCSC" "C1981952" (at 0 0 0) (effects (font (size 1.27 1.27)) (hide yes))) (property "Assembly" "FACTORY" (at 0 0 0) (effects (font (size 1.27 1.27)) (hide yes))))
+(symbol (lib_id "Device:D_Zener") (at 342.9 55.88 0) (unit 1) (in_bom yes) (on_board yes) (dnp no) (property "Reference" "D103" (at 337.82 46.99 0) (effects (font (size 1.27 1.27)) (justify left))) (property "Value" "SMCJ24A /TVS" (at 337.82 49.53 0) (effects (font (size 1.27 1.27)) (justify left))) (property "Footprint" "RevB:D_SMC_RVB22_D103" (at 0 0 0) (effects (font (size 1.27 1.27)) (justify left) hide)) (property "Datasheet" "~" (at 0 0 0) (effects (font (size 1.27 1.27)) (justify left) hide)) (property "MPN" "SMCJ24AHE3_A/H" (at 0 0 0) (effects (font (size 1.27 1.27)) (justify left) hide)) (property "Qualification" "VERIFIED component selection; qualification/productization/SELECTED_COMPONENTS.json; physical acceptance separate" (at 0 0 0) (effects (font (size 1.27 1.27)) (justify left) hide)) (pin "1") (pin "2") (instances (project "GR86_CCA_RevB" (path "/4108b523-946e-532e-b734-a3b8d9b0fa0b/33d5571c-9bbc-5869-9406-ade8bba2c66d" (reference "D103") (unit 1)))) (property "Manufacturer" "Vishay" (at 0 0 0) (effects (font (size 1.27 1.27)) (hide yes))) (property "LCSC" "C1981952" (at 0 0 0) (effects (font (size 1.27 1.27)) (hide yes))) (property "Assembly" "FACTORY" (at 0 0 0) (effects (font (size 1.27 1.27)) (hide yes))))
 (wire (pts (xy 38.1 105.41) (xy 38.1 100.33)) (stroke (width 0) (type default)))
 (global_label "REV_BLOCKED_12V" (shape bidirectional) (at 38.1 100.33 0) (effects (font (size 1.0 1.0)) (justify left)) (property "Intersheetrefs" "${INTERSHEET_REFS}" (at 38.1 100.33 0) (effects (font (size 1.27 1.27)) (justify left) hide)))
