File: docs/engineering/rvb22/candidate/cad/Power_5V.kicad_sch (KiCad schematic)
At the start: 23 parts, among them U121 LM5164DDAR

Commit message: fix(cca): reconcile controlled footprint variants and retain coupled thermal redlines
Parts:
- L121: footprint RevB:Coilcraft_MSS1246T_12x12 -> RevB:Coilcraft_MSS1246T_12x12_RVB22_L121
