File: docs/engineering/rvb22/candidate/cad/Vehicle_Interconnect.kicad_sch (KiCad schematic)
At the start: 1 part

Commit message: fix(cca): reconcile controlled footprint variants and retain coupled thermal redlines
Parts:
- F1: footprint RevB:Molex_Micro-Fit_3.0_43045-1200_2x06_P3.00mm_Horizontal -> RevB:Molex_Micro-Fit_3.0_43045-1200_2x06_P3.00mm_Horizontal_RVB22_F1
