File: docs/engineering/rvb22/candidate/cad/ESP32.kicad_sch (KiCad schematic)
At the start: 13 parts, among them U201 ESP32-S3-WROOM-1-N8R2, U202 TPS3808G33-Q1 3.07V RESET

Commit message: fix(cca): reconcile controlled footprint variants and retain coupled thermal redlines
Parts:
- C205: footprint RevB:C_0603_1608Metric -> RevB:C_0603_1608Metric_RVB22_C205
- R203: footprint RevB:R_0603_1608Metric -> RevB:R_0603_1608Metric_RVB22_R203
- U201: footprint RevB:ESP32-S3-WROOM-1 -> RevB:ESP32-S3-WROOM-1_RVB22_U201

Commit message: RVB22 I13: trial denser ESP thermal vias and retain failed thermal evidence
Parts:
- U201: footprint RevB:ESP32-S3-WROOM-1_RVB22_U201 -> RevB:ESP32-S3-WROOM-1_RVB22_U201_TH48
Changed lines of the file:
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@@
 (wire (pts (xy 86.36 124.46) (xy 81.28 124.46)) (stroke (width 0) (type default)))
 (global_label "GPS_PPS_MCU" (shape bidirectional) (at 81.28 124.46 180) (effects (font (size 1.0 1.0)) (justify right)) (property "Intersheetrefs" "${INTERSHEET_REFS}" (at 81.28 124.46 0) (effects (font (size 1.27 1.27)) (justify left) hide)))
-(symbol (lib_id "RF_Module:ESP32-S3-WROOM-1") (at 101.6 101.6 0) (unit 1) (in_bom yes) (on_board yes) (dnp no) (property "Reference" "U201" (at 114.3 66.04 0) (effects (font (size 1.27 1.27)) (justify left))) (property "Value" "ESP32-S3-WROOM-1-N8R2" (at 114.3 68.58 0) (effects (font (size 1.27 1.27)) (justify left))) (property "Footprint" "RevB:ESP32-S3-WROOM-1_RVB22_U201" (at 0 0 0) (effects (font (size 1.27 1.27)) (justify left) hide)) (property "Datasheet" "https://www.espressif.com/sites/default/files/documentation/esp32-s3-wroom-1_wroom-1u_datasheet_en.pdf" (at 0 0 0) (effects (font (size 1.27 1.27)) (justify left) hide)) (property "MPN" "ESP32-S3-WROOM-1-N8R2" (at 0 0 0) (effects (font (size 1.27 1.27)) (justify left) hide)) (property "Qualification" "VERIFIED component selection; qualification/productization/SELECTED_COMPONENTS.json; physical acceptance separate" (at 0 0 0) (effects (font (size 1.27 1.27)) (justify left) hide)) (pin "1") (pin "10") (pin "11") (pin "12") (pin "13") (pin "14") (pin "15") (pin "16") (pin "17") (pin "18") (pin "19") (pin "2") (pin "20") (pin "21") (pin "22") (pin "23") (pin "24") (pin "25") (pin "26") (pin "27") (pin "28") (pin "29") (pin "3") (pin "30") (pin "31") (pin "32") (pin "33") (pin "34") (pin "35") (pin "36") (pin "37") (pin "38") (pin "39") (pin "4") (pin "40") (pin "41") (pin "5") (pin "6") (pin "7") (pin "8") (pin "9") (instances (project "GR86_CCA_RevB" (path "/4108b523-946e-532e-b734-a3b8d9b0fa0b/fe7b91e6-7649-5595-9466-78a891f274f0" (reference "U201") (unit 1)))) (property "Manufacturer" "Espressif" (at 0 0 0) (effects (font (size 1.27 1.27)) (hide yes))) (property "LCSC" "C2913204" (at 0 0 0) (effects (font (size 1.27 1.27)) (hide yes))) (property "Assembly" "FACTORY" (at 0 0 0) (effects (font (size 1.27 1.27)) (hide yes))))
+(symbol (lib_id "RF_Module:ESP32-S3-WROOM-1") (at 101.6 101.6 0) (unit 1) (in_bom yes) (on_board yes) (dnp no) (property "Reference" "U201" (at 114.3 66.04 0) (effects (font (size 1.27 1.27)) (justify left))) (property "Value" "ESP32-S3-WROOM-1-N8R2" (at 114.3 68.58 0) (effects (font (size 1.27 1.27)) (justify left))) (property "Footprint" "RevB:ESP32-S3-WROOM-1_RVB22_U201_TH48" (at 0 0 0) (effects (font (size 1.27 1.27)) (justify left) hide)) (property "Datasheet" "https://www.espressif.com/sites/default/files/documentation/esp32-s3-wroom-1_wroom-1u_datasheet_en.pdf" (at 0 0 0) (effects (font (size 1.27 1.27)) (justify left) hide)) (property "MPN" "ESP32-S3-WROOM-1-N8R2" (at 0 0 0) (effects (font (size 1.27 1.27)) (justify left) hide)) (property "Qualification" "VERIFIED component selection; qualification/productization/SELECTED_COMPONENTS.json; physical acceptance separate" (at 0 0 0) (effects (font (size 1.27 1.27)) (justify left) hide)) (pin "1") (pin "10") (pin "11") (pin "12") (pin "13") (pin "14") (pin "15") (pin "16") (pin "17") (pin "18") (pin "19") (pin "2") (pin "20") (pin "21") (pin "22") (pin "23") (pin "24") (pin "25") (pin "26") (pin "27") (pin "28") (pin "29") (pin "3") (pin "30") (pin "31") (pin "32") (pin "33") (pin "34") (pin "35") (pin "36") (pin "37") (pin "38") (pin "39") (pin "4") (pin "40") (pin "41") (pin "5") (pin "6") (pin "7") (pin "8") (pin "9") (instances (project "GR86_CCA_RevB" (path "/4108b523-946e-532e-b734-a3b8d9b0fa0b/fe7b91e6-7649-5595-9466-78a891f274f0" (reference "U201") (unit 1)))) (property "Manufacturer" "Espressif" (at 0 0 0) (effects (font (size 1.27 1.27)) (hide yes))) (property "LCSC" "C2913204" (at 0 0 0) (effects (font (size 1.27 1.27)) (hide yes))) (property "Assembly" "FACTORY" (at 0 0 0) (effects (font (size 1.27 1.27)) (hide yes))))
 (wire (pts (xy 193.04 57.15) (xy 193.04 52.07)) (stroke (width 0) (type default)))
 (global_label "+3V3" (shape bidirectional) (at 193.04 52.07 0) (effects (font (size 1.0 1.0)) (justify left)) (property "Intersheetrefs" "${INTERSHEET_REFS}" (at 193.04 52.07 0) (effects (font (size 1.27 1.27)) (justify left) hide)))
